File: MotorDriver.sch (EAGLE design)
At the start: 49 parts, among them IC3 STM32F071V8T6V8, J8 B4B-PH-K-S(LF)(SN), M0 VNH7100ASTR, M1 VNH7100ASTR, M2 VNH7100ASTR, M3 VNH7100ASTR, M4 VNH7100ASTR, M5 VNH7100ASTR, M6 VNH7100ASTR, M7 VNH7100ASTR, U1 ICE5LP1K-SG48ITR, X1 MINI-USB-UX60-MB-5S8

Commit message: Update MotorDriver.sch
updates
Parts:
- removed SPLASH-MEMORY: N25Q032A13ESE40G, N25Q032A13ESC40F:N25Q032A13ESE40G
- removed U10: (no value), microbuilder:LP2985SOT23
- added SV8: (no value), con-lstb:MA20-2
- added U2: N25Q032A13ESC40F, N25Q032A13ESC40FNew:N25Q032A13ESC40F
- added U3: (no value), microbuilder:LP2985SOT23
- renumbered EN2 to EN1
Connections:
- removed net N$24: J8.3
- removed net N$25: J8.4
- removed net PA0: M4.INA
- removed net PA10: M1.INA
- removed net PA11: M1.INB
- removed net PA12: M2.INA
- removed net PA13: M2.INB
- removed net PA14: M3.INA
- removed net PA15: M3.INB
- removed net PA2: M4.INB
- removed net PA3: M5.INA
- removed net PA4: M5.INB
- removed net PA8: M0.INA
- removed net PA9: M0.INB
- removed net PC6: M0.PWM
- removed net PC7: M1.PWM
- removed net PC8: M2.PWM
- removed net PC9: M3.PWM
- removed net PE10: M7.INA
- removed net PE11: M5.PWM
- removed net PE12: M7.INB
- removed net PE13: M6.PWM
- removed net PE14: M7.PWM
- removed net PE7: M6.INA
- removed net PE8: M6.INB
- removed net PE9: M4.PWM
- new net M0-A: IC3.PA8, M0.INA
- new net M0-B: IC3.PA9, M0.INB
- new net M0-PWM: IC3.PC6, M0.PWM
- new net M1-A: IC3.PA10, M1.INA
- new net M1-B: IC3.PA11, M1.INB
- new net M1-PWM: IC3.PC7, M1.PWM
- new net M2-A: IC3.PA12, M2.INA
- new net M2-B: IC3.PA13, M2.INB
- new net M2-PWM: IC3.PC8, M2.PWM
- new net M3-A: IC3.PA14, M3.INA
- new net M3-B: IC3.PA15, M3.INB
- new net M3-PWM: IC3.PC9, M3.PWM
- new net M4-A: IC3.PA0, M4.INA
- new net M4-B: IC3.PA2, M4.INB
- new net M4-PWM: IC3.PE9, M4.PWM
- new net M5-A: IC3.PA3, M5.INA
- new net M5-B: IC3.PA4, M5.INB
- new net M5-PWM: IC3.PE11, M5.PWM
- new net M6-A: IC3.PE7, M6.INA
- new net M6-B: IC3.PE8, M6.INB
- new net M6-PWM: IC3.PE13, M6.PWM
- new net M7-A: IC3.PE10, M7.INA
- new net M7-B: IC3.PE12, M7.INB
- new net M7-PWM: IC3.PE14, M7.PWM
- new net RPI-BUSY: IC3.PB2, SV8.15
- new net RPI-CLK: IC3.PB13, SV8.23
- new net RPI-CS: IC3.PB12, SV8.29
- new net RPI-MISO: IC3.PB14, SV8.21
- new net RPI-MOSI: IC3.PB15, SV8.19
- new net RPI-READY: IC3.PB3, SV8.13
- new net RPI-STATUS: IC3.PB9, SV8.11
- new net RPI-USART-RX: IC3.PD10, SV8.10
- new net RPI-USART-TX: IC3.PD9, SV8.8
- net EN2-A: now also J8.3
- net EN2-B: now also J8.4

Commit message: Update MotorDriver.sch
updated-7/31
Parts:
- added C11, C12, C21, C22, C30, C31: 22UF-1210-16V-20%, SparkFun-Capacitors:22UF-1210-16V-20%
- added C13, C23, C32: GRM1552C1E220JA01-22pf, microbuilder:CAP_CERAMIC0402
- added C14, C18, C26, C27, C8, C9: 0.1uF, SparkFun-Capacitors:0.1UF-0603-25V-(+80/-20%)
- added C15: 20uF, SparkFun-Capacitors:10UF-1210-50V-20%
- added C16, C24, C33: GRM155B11H332KA01J-3300pf, microbuilder:CAP_CERAMIC0402
- added C17, C25, C34: 1.0uF, SparkFun-Capacitors:1.0UF-0603-16V-10%
- added C19, C20, C28, C29: 10uF, SparkFun-Capacitors:10UF-1210-50V-20%
- added C35, C36, C37, C5, C6, C7: 10uF, SparkFun-Capacitors:10UF-0603-6.3V-20%
- added CR1-LINEAR-POWER1, CR1-LINEAR-POWER2, CR2-LINEAR-REGULATOR: LD1085D2T33R, LD1085D2T33:LD1085D2T33R
- added L1, L2, L3: FDSD0518-H-3R3M=P3, FDSD0518-H-3R3M_P3:FDSD0518-H-3R3M=P3
- added Q2: 20V/4.2A/52mΩ/1.4W, SparkFun-DiscreteSemi:MOSFET_PCH-DMG2305UX-7
- added R12: 10k, SparkFun-Resistors:10KOHM-0402-1/16W-1%
- added R13: 47K, SparkFun-Resistors:10KOHM-0402-1/16W-1%
- added R14, R19, R5: MCR01MZPJ000, MCR01MZPJ000:MCR01MZPJ000
- added R15, R18, R20, R23, R6, R9: MCR01MZPF1801, MCR01MZPF1801:MCR01MZPF1801
- added R16, R21, R7: MCR01MZPF1203, MCR01MZPF1203:MCR01MZPF1203
- added R17, R22, R8: MCR01MZPF2202, MCR01MZPF2202:MCR01MZPF2202
- added R24, R25, R26, R27: 120ohms, SparkFun-Resistors:124KOHM
- added SWITCHING-REGULATOR, U4: BD9D323QWZ-E2, BD9D323QWZ:BD9D323QWZ-E2
- added U3-PROTECTION-CIRCUIT: MMDT5401-7-F, MMDT5401:MMDT5401-7-F
- U3: value (none) -> BD9D323QWZ-E2; device microbuilder:LP2985SOT23 -> BD9D323QWZ:BD9D323QWZ-E2
Connections:
- new net EN-PWR: EN3.1, EN4.1, EN5.1, EN6.1, EN7.1, J8.1
- new net N$13: C16.P$1, SWITCHING-REGULATOR.SS
- new net N$14: C13.P$1, R5.1, R6.1
- new net N$15: R6.2, R7.1
- new net N$16: C13.P$2, R7.2, R8.2, R9.2, SWITCHING-REGULATOR.FB
- new net N$17: C17.1, SWITCHING-REGULATOR.VREG
- new net N$18: C14.1, L2.2, R9.1, SWITCHING-REGULATOR.SW
- new net N$20: C18.2, U3.BOOT
- new net N$21: C23.P$1, R14.1, R15.1
- new net N$22: Q2.G, R13.1, U3-PROTECTION-CIRCUIT.E2
- new net N$23: R12.2, U3-PROTECTION-CIRCUIT.B1, U3-PROTECTION-CIRCUIT.C2, U3-PROTECTION-CIRCUIT.E1
- new net N$24: R15.2, R16.1
- new net N$25: C18.1, L1.2, R18.1, U3.SW
- new net N$26: C24.P$1, U3.SS
- new net N$27: C25.1, U3.VREG
- new net N$28: C23.P$2, R16.2, R17.2, R18.2, U3.FB
- new net N$29: C27.2, U4.BOOT
- new net N$30: C32.P$1, R19.1, R20.1
- new net N$31: R20.2, R21.1
- new net N$32: C27.1, L3.2, R23.1, U4.SW
- new net N$33: C33.P$1, U4.SS
- new net N$34: C34.1, U4.VREG
- new net N$35: C32.P$2, R21.2, R22.2, R23.2, U4.FB
- new net N$36: CR1-LINEAR-POWER1.GROUND, R24.1, R25.2
- new net N$37: CR1-LINEAR-POWER2.GROUND, R26.1, R27.2
- new net N$4: C14.2, SWITCHING-REGULATOR.BOOT
- new net RPI: Q2.S, U3-PROTECTION-CIRCUIT.B2
- new net SERVO-6V: C35.1, C36.1, CR1-LINEAR-POWER1.OUTPUT, CR1-LINEAR-POWER2.OUTPUT, R24.2, R26.2
- new net V-IN-12V: C15.1, C19.1, C20.1, C26.1, C28.1, C29.1, C37.1, C5.1, C7.1, C8.1, C9.1, CR1-LINEAR-POWER1.INPUT, CR1-LINEAR-POWER2.INPUT, CR2-LINEAR-REGULATOR.INPUT, M0.VCC, M1.VCC, M2.VCC, M3.VCC, M4.VCC, M5.VCC, M6.VCC, M7.VCC, SWITCHING-REGULATOR.EN, SWITCHING-REGULATOR.VIN, U3.EN, U3.VIN, U4.EN, U4.VIN
- new net VCC-5V: C11.1, C12.1, C21.1, C22.1, C30.1, C31.1, C6.1, CR2-LINEAR-REGULATOR.OUTPUT, L1.1, L2.1, L3.1, Q2.D, R14.2, R19.2, R5.2, U3-PROTECTION-CIRCUIT.C1
- net EN_PWR: no longer EN3.2, EN4.2, EN5.2, EN6.2, EN7.2, J8.2
- net GND: now also C11.2, C12.2, C15.2, C16.P$2, C17.2, C19.2, C20.2, C21.2, C22.2, C24.P$2, C25.2, C26.2, C28.2, C29.2, C30.2, C31.2, C33.P$2, C34.2, C35.2, C36.2, C37.2, C5.2, C6.2, C7.2, C8.2, C9.2, CR2-LINEAR-REGULATOR.GROUND, EN3.2, EN4.2, EN5.2, EN6.2, EN7.2, IC3.VSS@4, J8.2, M0.GNDA, M0.GNDB, M1.GNDA, M1.GNDB, M2.GNDA, M2.GNDB, M3.GNDA, M3.GNDB, M4.GNDA, M4.GNDB, M5.GNDA, M5.GNDB, M6.GNDA, M6.GNDB, M7.GNDA, M7.GNDB, R12.1, R13.2, R17.1, R22.1, R25.1, R27.1, R8.1, SV8.6, SWITCHING-REGULATOR.GND, U3.GND, U4.GND; no longer EN3.1, EN4.1, EN5.1, EN6.1, EN7.1, J8.1

Commit message: added brd file
Parts:
- removed C20, C29: 10uF, SparkFun-Capacitors:10UF-1210-50V-20%
- removed CR2-LINEAR-REGULATOR: LD1085D2T33R, LD1085D2T33:LD1085D2T33R
- removed R12: 10k, SparkFun-Resistors:10KOHM-0402-1/16W-1%
- removed R13: 47K, SparkFun-Resistors:10KOHM-0402-1/16W-1%
- removed SV0, SV1, SV2, SV3, SV4, SV5, SV6, SV7: (no value), con-lstb:MA03-1
- removed SWITCHING-REGULATOR: BD9D323QWZ-E2, BD9D323QWZ:BD9D323QWZ-E2
- removed U3-PROTECTION-CIRCUIT: MMDT5401-7-F, MMDT5401:MMDT5401-7-F
- added C41, C45, C48: 10nF, SparkFun-Capacitors:10NF-0603-50V-10%
- added C42, C43, C46, C47: 100nF, SparkFun-Capacitors:10NF-0603-50V-10%
- added C44: 0.1uF, SparkFun-Capacitors:0.1UF-0603-25V-(+80/-20%)
- added C49, C50, C51, C52: 1.0uF, SparkFun-Capacitors:1.0UF-0603-16V-10%
- added J0, J1, J2, J3, J4, J5, J6, J7: (no value), con-lstb:MA03-1
- added J11: B4B-PH-K-S(LF)(SN), B4B-PH-K-S_LF__SN_:B4B-PH-K-S(LF)(SN)
- added J26: XT30PWXT30PW, XT30PW:XT30PWXT30PW
- added J28: (no value), con-lstb:MA04-2
- added J29: (no value), SparkFun-Connectors:CONN_02
- added JTAG: CORTEX_JTAG_DEBUG_SMD, SparkFun-Connectors:CORTEX_JTAG_DEBUG_SMD
- added R10, R11, R28, R29, R30, R31: 10k, SparkFun-Resistors:10KOHM-0603-1/10W-1%
- added R4: 100, SparkFun-Resistors:100OHM-0603-1/4W-5%
- added U5: MMDT5401-7-F, MMDT5401:MMDT5401-7-F
- added U6: BD9D323QWZ-E2, BD9D323QWZ:BD9D323QWZ-E2
- added U7: MIC5504-3.3YM5-TR, MIC5504-3.3YM5-TR:MIC5504-3.3YM5-TR
- added U8: MIC5365-1.2YC5-TR, MIC5365-1.2YC5:MIC5365-1.2YC5-TR
- added U9: LD1085D2T33R, LD1085D2T33:LD1085D2T33R
- added Y1: ECS-TXO-2520-33-160-AN-TR, ECS-TXO-2520-33-160-AN-TR:ECS-TXO-2520-33-160-AN-TR
- C19, C28: value 10uF -> 20uF
- J8: value B4B-PH-K-S(LF)(SN) -> (none); device B4B-PH-K-S_LF__SN_:B4B-PH-K-S(LF)(SN) -> con-lstb:MA03-2
- renumbered CR1-LINEAR-POWER1 to U10, CR1-LINEAR-POWER2 to U11, EN0 to J9, EN1 to J10, EN3 to J12, EN4 to J13, EN5 to J14, EN6 to J15, EN7 to J16, SV8 to J17, XA10 to J24, XA11 to J20, XA12 to J21, XA13 to J22, XA14 to J23, XA15 to J25, XA16 to J18, XA9 to J19
Connections:
- net CRYSTAL0-OUT renamed CRYSTAL0_OUT
- net CRYSTAL1-IN renamed CRYSTAL1_IN
- net CRYSTAL1-OUT renamed CRYSTAL1_OUT
- net CRYTAL0-IN renamed CRYTAL0_IN
- net M0-A renamed M0_A
- net M0-B renamed M0_B
- net M0-PWM renamed M0_PWM
- net M1-A renamed M1_A
- net M1-B renamed M1_B
- net M1-PWM renamed M1_PWM
- net M2-A renamed M2_A
- net M2-PWM renamed M2_PWM
- net M3-B renamed M3_B
- net M3-PWM renamed M3_PWM
- net M4-A renamed M4_A
- net M4-B renamed M4_B
- net M4-PWM renamed M4_PWM
- net M5-A renamed M5_A
- net M5-B renamed M5_B
- net M5-PWM renamed M5_PWM
- net M6-A renamed M6_A
- net M6-B renamed M6_B
- net M6-PWM renamed M6_PWM
- net M7-A renamed M7_A
- net M7-B renamed M7_B
- net M7-PWM renamed M7_PWM
- net OUT0-A renamed OUT0_A
- net OUT0-B renamed OUT0_B
- net OUT1-A renamed OUT1_A
- net OUT1-B renamed OUT1_B
- net OUT2-A renamed OUT2_A
- net OUT2-B renamed OUT2_B
- net OUT3-A renamed OUT3_A
- net OUT3-B renamed OUT3_B
- net OUT4-A renamed OUT4_A
- net OUT4-B renamed OUT4_B
- net OUT5-A renamed OUT5_A
- net OUT5-B renamed OUT5_B
- net OUT6-A renamed OUT6_A
- net OUT6-B renamed OUT6_B
- net OUT7-A renamed OUT7_A
- net OUT7-B renamed OUT7_B
- net RPI-BUSY renamed RPI_BUSY
- net RPI-CLK renamed RPI_CLK
- net RPI-CS renamed RPI_CS
- net RPI-MISO renamed RPI_MISO
- net RPI-MOSI renamed RPI_MOSI
- net RPI-READY renamed RPI_READY
- net RPI-STATUS renamed RPI_STATUS
- net RPI-USART-RX renamed RPI_USART_RX
- net RPI-USART-TX renamed RPI_USART_TX
- removed net EN-PWR: J12.1, J13.1, J14.1, J15.1, J16.1, J8.1
- removed net EN_PWR: J10.2, J9.2
- removed net M2-B: IC3.PA13, M2.INB
- removed net M3-A: IC3.PA14, M3.INA
- removed net N$10: SV5.2
- removed net N$11: SV6.2
- removed net N$12: SV7.2
- removed net N$8: SV3.2
- removed net N$9: SV4.2
- removed net RPI: Q2.S, U3-PROTECTION-CIRCUIT.B2
- removed net SERVO-6V: C35.1, C36.1, R24.2, R26.2, U10.OUTPUT, U11.OUTPUT
- removed net SV_PWR: SV0.2
- removed net V-IN-12V: C15.1, C19.1, C20.1, C26.1, C28.1, C29.1, C37.1, C5.1, C7.1, C8.1, C9.1, CR2-LINEAR-REGULATOR.INPUT, M0.VCC, M1.VCC, M2.VCC, M3.VCC, M4.VCC, M5.VCC, M6.VCC, M7.VCC, SWITCHING-REGULATOR.EN, SWITCHING-REGULATOR.VIN, U10.INPUT, U11.INPUT, U3.EN, U3.VIN, U4.EN, U4.VIN
- removed net VCC-5V: C11.1, C12.1, C21.1, C22.1, C30.1, C31.1, C6.1, CR2-LINEAR-REGULATOR.OUTPUT, L1.1, L2.1, L3.1, Q2.D, R14.2, R19.2, R5.2, U3-PROTECTION-CIRCUIT.C1
- new net EXTENAL_CLK: U1.IOT_46B_G0
- new net EXTERNAL_CLK: Y1.OUTPUT
- new net FLASH_CLK: J28.1, J8.1, R10.1, U1.IOB_34A_SPI_SCK, U2.C
- new net FLASH_CS: J28.2, J8.2, R29.1, U1.IOB_35B_SPI_CSN, U2.S-
- new net FLASH_HOLD: J28.7, R11.1, U2.HOLD-/DQ3
- new net FLASH_MISO: J28.3, J8.3, U1.IOB_32A_SPI_SO, U2.DQ1
- new net FLASH_MOSI: J28.4, J8.4, U1.IOB_33B_SPI_SI, U2.DQ0
- new net FLASH_WP: J28.8, R28.1, U2.W-/VPP/DQ2
- new net FPGA_CDONE: IC3.PE5, U1.CDONE
- new net FPGA_CRESET_B: IC3.PE4, U1.CRESET_B
- new net JTAG_RESET: IC3.NRST, JTAG.!RESET
- new net JTAG_SWDCLK: IC3.PA14, JTAG.SWDCLK/TCK
- new net JTAG_SWDIO: IC3.PA13, JTAG.SWDIO/TMS
- new net M2_B: IC3.PE3, M2.INB
- new net M3_A: IC3.PE2, M3.INA
- new net N$19: JTAG.NC/TDI
- new net N$38: JTAG.SWO/TDO
- new net N$5: C45.1, C47.1, R4.1, U1.VCCPLL
- new net RPI_5V: J17.2, J17.4, J29.1, Q2.S, U5.B2
- new net SERVO_A_6V: C21.1, C22.1, C35.1, J0.2, J1.2, J2.2, J3.2, L1.1, R14.2, R24.2, U10.OUTPUT
- new net SERVO_B_6V: C30.1, C31.1, C36.1, J4.2, J5.2, J6.2, J7.2, L3.1, R19.2, R26.2, U11.OUTPUT
- new net VCC_12V: C15.1, C19.1, C26.1, C28.1, C37.1, C5.1, C7.1, C8.1, C9.1, J26.+, M0.VCC, M1.VCC, M2.VCC, M3.VCC, M4.VCC, M5.VCC, M6.VCC, M7.VCC, U10.INPUT, U11.INPUT, U3.EN, U3.VIN, U4.EN, U4.VIN, U6.EN, U6.VIN, U9.INPUT
- new net VCC_1_2V: C41.1, C52.1, R4.2, U1.VCC, U8.VOUT
- new net VCC_3.3V: C41.2, C42.1, C42.2, C43.1, C43.2, C44.1, C45.2, C46.1, C46.2, C47.2, C48.1, C48.2, C50.1, C51.1, IC3.VBAT, IC3.VDD@1, IC3.VDD@2, IC3.VDD@4, IC3.VDDA, IC3.VDDIO2, J10.2, J11.2, J12.2, J13.2, J14.2, J15.2, J16.2, J17.17, J28.5, J8.5, J9.2, JTAG.VCC, R10.2, R11.2, R28.2, R29.2, U1.SPI_VCCIO1, U1.VCCIO_0, U1.VCCIO_2, U1.VPP_2V5, U2.VCC, U7.NC, U7.VOUT, U8.EN, U8.VIN, Y1.VDD
- new net VCC_5V: C11.1, C12.1, C6.1, L2.1, Q2.D, R5.2, U5.C1, U7.VIN, U9.OUTPUT
- net EN2-A: now also J11.3; no longer J8.3
- net EN2-B: now also J11.4; no longer J8.4
- net GND: now also C44.2, C49.2, C50.2, C51.2, C52.2, IC3.BOOT0, IC3.VSS@1, IC3.VSS@2, IC3.VSS@3, IC3.VSSA, J0.3, J1.3, J11.1, J12.1, J13.1, J14.1, J15.1, J16.1, J17.14, J17.20, J17.25, J17.30, J17.34, J17.39, J17.9, J2.3, J26.-, J28.6, J29.2, J3.3, J4.3, J5.3, J6.3, J7.3, J8.6, JTAG.GND@3, JTAG.GND@5, JTAG.GNDDTCT, R30.1, R31.1, U2.VSS, U6.GND, U7.GND, U8.GND, U9.GROUND, Y1.GND; no longer C20.2, C29.2, CR2-LINEAR-REGULATOR.GROUND, J12.2, J13.2, J14.2, J15.2, J16.2, J8.2, R12.1, R13.2, SV0.3, SV1.3, SV2.3, SV3.3, SV4.3, SV5.3, SV6.3, SV7.3, SWITCHING-REGULATOR.GND
- net N$13: now also U6.SS; no longer SWITCHING-REGULATOR.SS
- net N$16: now also U6.FB; no longer SWITCHING-REGULATOR.FB
- net N$17: now also U6.VREG; no longer SWITCHING-REGULATOR.VREG
- net N$18: now also U6.SW; no longer SWITCHING-REGULATOR.SW
- net N$22: now also R31.2, U5.E2; no longer R13.1, U3-PROTECTION-CIRCUIT.E2
- net N$23: now also R30.2, U5.B1, U5.C2, U5.E1; no longer R12.2, U3-PROTECTION-CIRCUIT.B1, U3-PROTECTION-CIRCUIT.C2, U3-PROTECTION-CIRCUIT.E1
- net N$4: now also U6.BOOT; no longer SWITCHING-REGULATOR.BOOT
- net N$6: now also J17.1; no longer SV1.2
- net N$7: now also C49.1, U7.EN; no longer SV2.2
- net SV0_PWM0: now also J0.1; no longer SV0.1
- net SV1_PWM1: now also J1.1; no longer SV1.1
- net SV2_PWM2: now also J2.1; no longer SV2.1
- net SV3_PWM3: now also J3.1; no longer SV3.1
- net SV4_PWM4: now also J4.1; no longer SV4.1
- net SV5_PWM5: now also J5.1; no longer SV5.1
- net SV6_PWM6: now also J6.1; no longer SV6.1
- net SV7_PWM7: now also J7.1; no longer SV7.1

Commit message: Update
Parts:
- removed J29: (no value), SparkFun-Connectors:CONN_02
Connections:
- removed net CRYTAL0_IN: IC3.PC14-OSC32_IN
- removed net EXTENAL_CLK: U1.IOT_46B_G0
- removed net N$19: JTAG.NC/TDI
- removed net N$38: JTAG.SWO/TDO
- removed net N$5: C45.1, C47.1, R4.1, U1.VCCPLL
- removed net N$6: J17.1
- new net FPGA_FLASH_CLK: J28.1, U1.IOB_34A_SPI_SCK
- new net FPGA_FLASH_CS: J28.5, U1.IOB_35B_SPI_CSN
- new net FPGA_FLASH_MISO: J28.3, U1.IOB_32A_SPI_SO
- new net FPGA_FLASH_MOSI: J28.7, U1.IOB_33B_SPI_SI
- net CRYSTAL0-IN: now also IC3.PC14-OSC32_IN
- net EXTERNAL_CLK: now also U1.IOT_46B_G0
- net FLASH_CLK: now also J28.2; no longer J28.1, U1.IOB_34A_SPI_SCK
- net FLASH_CS: now also J28.6; no longer J28.2, U1.IOB_35B_SPI_CSN
- net FLASH_HOLD: no longer J28.7
- net FLASH_MISO: now also J28.4; no longer J28.3, U1.IOB_32A_SPI_SO
- net FLASH_MOSI: now also J28.8; no longer J28.4, U1.IOB_33B_SPI_SI
- net FLASH_WP: no longer J28.8
- net FPGA_CDONE: now also IC3.PC5; no longer IC3.PE5
- net FPGA_CRESET_B: now also IC3.PC4; no longer IC3.PE4
- net FPGA_CS: now also IC3.PB0; no longer IC3.PA1
- net GND: now also C41.2, C42.2, C43.2, C45.2, C46.2, C47.2, C48.2; no longer J28.6, J29.2
- net M0_A: now also IC3.PD14; no longer IC3.PA8
- net M0_B: now also IC3.PD15; no longer IC3.PA9
- net M1_A: now also IC3.PD12; no longer IC3.PA10
- net M1_B: now also IC3.PD13; no longer IC3.PA11
- net M2_A: now also IC3.PA8; no longer IC3.PA12
- net M2_B: now also IC3.PA9; no longer IC3.PE3
- net M3_A: now also IC3.PA10; no longer IC3.PE2
- net M3_B: now also IC3.PA11; no longer IC3.PA15
- net M4_A: now also IC3.PB2; no longer IC3.PA0
- net M4_B: now also IC3.PB1; no longer IC3.PA2
- net M5_A: now also IC3.PE8; no longer IC3.PA3
- net M5_B: now also IC3.PE7; no longer IC3.PA4
- net M6_A: now also IC3.PE12; no longer IC3.PE7
- net M6_B: now also IC3.PE10; no longer IC3.PE8
- net M7_A: now also IC3.PB10; no longer IC3.PE10
- net M7_B: now also IC3.PE15; no longer IC3.PE12
- net RPI_5V: no longer J29.1
- net RPI_BUSY: now also IC3.PB11; no longer IC3.PB2
- net RPI_READY: now also IC3.PD11; no longer IC3.PB3
- net RPI_STATUS: now also IC3.PD8; no longer IC3.PB9
- net VCC_1_2V: now also C45.1, C47.1, R4.1, U1.VCCPLL
- net VCC_3.3V: no longer C41.2, C42.2, C43.2, C45.2, C46.2, C47.2, C48.2, J17.17, J28.5

Commit message: update
Parts:
- removed J28: (no value), con-lstb:MA04-2
- removed Q0, Q1: (no value), crystal:CRYSTALHC49S
- added C20, C29, C38, C53, C54, C55: 22PF-0603-50V-5%, SparkFun-Capacitors:22PF-0603-50V-5%
- added R12, R13, R32, R33: 100, SparkFun-Resistors:100OHM-0603-1/4W-5%
- added Y2: 32.768kHz, SparkFun-Clocks:CRYSTAL-32.768KHZSMD-3.2X1.5
- added Y4: CRYSTAL-GROUNDEDSMD-3.2X2.5, SparkFun-Clocks:CRYSTAL-GROUNDEDSMD-3.2X2.5
- C11, C12, C21, C22, C30, C31: value 22UF-1210-16V-20% -> GRM32ER61E226KE15L; device SparkFun-Capacitors:22UF-1210-16V-20% -> GRM32ER61E226KE15L:GRM32ER61E226KE15L
Connections:
- new net 3.3V: C20.2, IC3.VDDIO2
- new net CRYSTAL0_IN: C4.1, Y2.2
- new net N$5: C53.2, IC3.VDD@2
- net CRYSTAL0-IN: no longer C4.1, Q1.2
- net CRYSTAL0_OUT: now also Y2.1; no longer Q1.1
- net CRYSTAL1_IN: now also Y4.2; no longer Q0.2
- net CRYSTAL1_OUT: now also Y4.1; no longer Q0.1
- net FLASH_CLK: no longer J28.2
- net FLASH_CS: no longer J28.6
- net FLASH_MISO: no longer J28.4
- net FLASH_MOSI: no longer J28.8
- net FPGA_CLK: now also R13.2
- net FPGA_CS: now also R12.2
- net FPGA_FLASH_CLK: now also R13.1; no longer J28.1
- net FPGA_FLASH_CS: now also R12.1; no longer J28.5
- net FPGA_FLASH_MISO: now also R32.1; no longer J28.3
- net FPGA_FLASH_MOSI: now also R33.1; no longer J28.7
- net FPGA_MISO: now also R32.2
- net FPGA_MOSI: now also R33.2
- net GND: now also C20.1, C29.1, C38.1, C53.1, C54.1, C55.2, U4.EPAD, Y4.3
- net VCC_3.3V: now also C29.2, C38.2, C54.2, C55.1; no longer IC3.VDD@2, IC3.VDDIO2
Other:
- moved on the sheet: C11, C12, C21, C22, C30, C31

Commit message: update
Connections:
- net GND: now also U3.EPAD, U6.EPAD
Changed lines of the file:
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@@
 <part name="C55" library="SparkFun-Capacitors" deviceset="22PF" device="-0603-50V-5%" value=""/>
 <part name="GND88" library="SparkFun-PowerSymbols" deviceset="GND" device=""/>
+<part name="GND89" library="SparkFun-PowerSymbols" deviceset="GND" device=""/>
+<part name="GND90" library="SparkFun-PowerSymbols" deviceset="GND" device=""/>
 </parts>
 <sheets>
@@
 <attribute name="VALUE" x="172.72" y="-66.294" size="1.778" layer="96" align="top-center"/>
 </instance>
+<instance part="GND89" gate="1" x="-2.54" y="53.34" smashed="yes">
+<attribute name="VALUE" x="-2.54" y="53.086" size="1.778" layer="96" align="top-center"/>
+</instance>
 </instances>
 <busses>
@@
 <wire x1="172.72" y1="-40.64" x2="172.72" y2="-63.5" width="0.1524" layer="91"/>
 </segment>
+<segment>
+<pinref part="U3" gate="A" pin="EPAD"/>
+<wire x1="-27.94" y1="78.74" x2="-2.54" y2="78.74" width="0.1524" layer="91"/>
+<wire x1="-2.54" y1="78.74" x2="-2.54" y2="55.88" width="0.1524" layer="91"/>
+<pinref part="GND89" gate="1" pin="GND"/>
+</segment>
 </net>
 <net name="N$20" class="0">
@@
 <attribute name="VALUE" x="160.02" y="45.974" size="1.778" layer="96" align="bottom-center"/>
 </instance>
+<instance part="GND90" gate="1" x="22.86" y="22.86" smashed="yes">
+<attribute name="VALUE" x="22.86" y="22.606" size="1.778" layer="96" align="top-center"/>
+</instance>
 </instances>
 <busses>
@@
 <wire x1="-83.82" y1="-63.5" x2="-83.82" y2="-86.36" width="0.1524" layer="91"/>
 </segment>
+<segment>
+<pinref part="U6" gate="A" pin="EPAD"/>
+<wire x1="0" y1="48.26" x2="22.86" y2="48.26" width="0.1524" layer="91"/>
+<wire x1="22.86" y1="48.26" x2="22.86" y2="25.4" width="0.1524" layer="91"/>
+<pinref part="GND90" gate="1" pin="GND"/>
+</segment>
 </net>

Commit message: update
Connections:
- removed net CRYSTAL0-IN: IC3.PC14-OSC32_IN
- removed net N$5: C53.2, IC3.VDD@2
- new net N$8: C45.1, C47.1, R4.1, U1.VCCPLL
- net CRYSTAL0_IN: now also IC3.PC14-OSC32_IN
- net VCC_1_2V: no longer C45.1, C47.1, R4.1, U1.VCCPLL
- net VCC_3.3V: now also C53.2, IC3.VDD@2
Other:
- moved on the sheet: C11, C12, C45

Commit message: update
Parts:
- added SV1: (no value), con-lstb:MA04-2
- C42, C45, C47: device SparkFun-Capacitors:10NF-0603-50V-10% -> SparkFun-Capacitors:1.0UF-0402T-16V-10%
- R4: device SparkFun-Resistors:100OHM-0603-1/4W-5% -> SparkFun-Resistors:2.2KOHM-0402-1/16W-1%
Connections:
- net FLASH_CLK: now also SV1.4
- net FLASH_CS: now also SV1.8
- net FLASH_MISO: now also SV1.6
- net FLASH_MOSI: now also SV1.2
- net FPGA_FLASH_CLK: now also SV1.3
- net FPGA_FLASH_CS: now also SV1.7
- net FPGA_FLASH_MISO: now also SV1.5
- net FPGA_FLASH_MOSI: now also SV1.1
