File: MotorDriver.sch (EAGLE design)
At the start: 145 parts, among them IC3 STM32F071V8T6V8, J10 B4B-PH-K-S(LF)(SN), J11 B4B-PH-K-S(LF)(SN), J12 B4B-PH-K-S(LF)(SN), J13 B4B-PH-K-S(LF)(SN), J14 B4B-PH-K-S(LF)(SN), J15 B4B-PH-K-S(LF)(SN), J16 B4B-PH-K-S(LF)(SN), J18 B2P-VH(LF)(SN), J19 B2P-VH(LF)(SN), J20 B2P-VH(LF)(SN), J21 B2P-VH(LF)(SN), J22 B2P-VH(LF)(SN), J23 B2P-VH(LF)(SN), J24 B2P-VH(LF)(SN), J25 B2P-VH(LF)(SN), J26 XT30PWXT30PW, J9 B4B-PH-K-S(LF)(SN), M0 VNH7100ASTR, M1 VNH7100ASTR, M2 VNH7100ASTR, M3 VNH7100ASTR, M4 VNH7100ASTR, M5 VNH7100ASTR, M6 VNH7100ASTR, M7 VNH7100ASTR, Q2 20V/4.2A/52mΩ/1.4W, U1 ICE5LP1K-SG48ITR, U10 LD1085D2T33R, U11 LD1085D2T33R, U2 N25Q032A13ESC40F, U3 BD9D323QWZ-E2, U4 BD9D323QWZ-E2, U5 MMDT5401-7-F, U6 BD9D323QWZ-E2, U7 MIC5504-3.3YM5-TR, U8 MIC5365-1.2YC5-TR, U9 LD1085D2T33R, X1 MINI-USB-UX60-MB-5S8, Y1 ECS-TXO-2520-33-160-AN-TR, Y2 32.768kHz, Y4 CRYSTAL-GROUNDEDSMD-3.2X2.5

Commit message: update
Parts:
- C1, C2, C3, C4: value 22pF -> 1.0uF; device SparkFun-Capacitors:22PF-0603-50V-5% -> SparkFun-Capacitors:1.0UF-0402T-16V-10%
- C20, C29, C38, C53, C54, C55: value 22PF-0603-50V-5% -> 1.0uF; device SparkFun-Capacitors:22PF-0603-50V-5% -> SparkFun-Capacitors:1.0UF-0402T-16V-10%
- C41, C48: value 10nF -> 1.0uF; device SparkFun-Capacitors:10NF-0603-50V-10% -> SparkFun-Capacitors:1.0UF-0402T-16V-10%
- C43, C46: value 100nF -> 1.0uF; device SparkFun-Capacitors:10NF-0603-50V-10% -> SparkFun-Capacitors:1.0UF-0402T-16V-10%
- C44: value 0.1uF -> 1.0uF; device SparkFun-Capacitors:0.1UF-0603-25V-(+80/-20%) -> SparkFun-Capacitors:1.0UF-0402T-16V-10%
Connections:
- new net LED1: D1.A, IC3.PD7
- new net LED2: D2.A, IC3.PB3
- new net LED3: D3.A, IC3.PB4
Other:
- moved on the sheet: D1, D2, D3, R1, R2, R3

Commit message: Adding Eagle Files
Parts:
- removed X1: MINI-USB-UX60-MB-5S8, con-hirose:MINI-USB-UX60-MB-5S8
- added C10, C39, C40, C56, C57, C58, C59, C60: 100uF, SparkFun-Capacitors:100UF-POLAR-25V-20%(ELEC)
- added C61: 120nF, SparkFun-Capacitors:1.0UF-0402T-16V-10%
- added C62: 6.8nF, SparkFun-Capacitors:1.0UF-0402T-16V-10%
- added C63, C64: 100nF, SparkFun-Capacitors:1.0UF-0402T-16V-10%
- added C65, C66: 1.0uF, SparkFun-Capacitors:1.0UF-0603-16V-10%
- added C67: 1.0uF, SparkFun-Capacitors:1.0UF-0402T-16V-10%
- added D4: (no value), SparkFun-LED:LED0603
- added H1, H2, H3, H4: MOUNT-HOLE3.6, holes:MOUNT-HOLE3.6
- added R34: 330, SparkFun-Resistors:330OHM-0603-1/10W-1%
- added R35, R36, R41, R42, R43: 47k, SparkFun-Resistors:2.2KOHM-0402T-1/16W-1%
- added R37: 10k, SparkFun-Resistors:2.2KOHM-0402T-1/16W-1%
- added R38, R39: 10k, SparkFun-Resistors:10KOHM-0603-1/10W-1%
- added R40: MCR01MZPF1801, MCR01MZPF1801:MCR01MZPF1801
- added U12: BNO055, BNO055:BNO055
- C35, C36, C37, C5, C6, C7: device SparkFun-Capacitors:10UF-0603-6.3V-20% -> SparkFun-Capacitors:10UF-0805-25V-10%
- R4: device SparkFun-Resistors:2.2KOHM-0402-1/16W-1% -> SparkFun-Resistors:2.2KOHM-0402T-1/16W-1%
Connections:
- removed net 3.3V: C20.2, IC3.VDDIO2
- new net GYRO_RESET: IC3.PB7, U12.NRESET
- new net I2C1_SCL: IC3.PB8, R35.1, U12.COM1
- new net I2C1_SDA: IC3.PB9, R36.1, U12.COM0
- new net INT: IC3.PB6, U12.INT
- new net N$10: C66.1, U8.NC
- new net N$11: C65.1, U7.NC
- new net N$12: J17.24, R41.1
- new net N$19: J17.26, R42.1
- new net N$38: J17.29, R43.2
- new net N$5: D4.C, R34.2
- new net N$6: R37.2, U12.NBOOT_LOAD_PIN
- new net N$9: C64.2, U12.CAP
- net FLASH_MISO: now also J8.4, U2.DQ0; no longer J8.3, U2.DQ1
- net FLASH_MOSI: now also J8.3, U2.DQ1; no longer J8.4, U2.DQ0
- net FPGA_CDONE: now also R39.1
- net FPGA_CRESET_B: now also C67.1, R38.1
- net GND: now also C10.-, C39.-, C40.-, C56.-, C57.-, C58.-, C59.-, C60.-, C61.1, C62.1, C63.1, C64.1, C65.2, C66.2, C67.2, R34.1, U12.COM2, U12.COM3, U12.GND, U12.GNDIO, U12.PIN15, U12.PIN16, U12.PS0, U12.PS1
- net N$7: now also R40.1
- net RPI_CS: now also R41.2, R42.2, R43.1; no longer J17.29
- net RPI_STATUS: now also IC3.PD10; no longer IC3.PD8
- net RPI_USART_RX: now also IC3.PD8; no longer IC3.PD10
- net VCC_12V: now also C10.+, C39.+, C40.+, C56.+, C57.+, C58.+, C59.+, C60.+
- net VCC_1_2V: now also R40.2
- net VCC_3.3V: now also C20.2, C61.2, C62.2, C63.2, D4.A, IC3.VDDIO2, R35.2, R36.2, R37.1, R38.2, R39.2, U12.VDD, U12.VDDIO; no longer C51.1, U7.NC, U8.EN, U8.VIN
- net VCC_5V: now also C51.1, U8.EN, U8.VIN
Other:
- moved on the sheet: C1, C2, C20, C3, C4, C49, C50, C51, C52, J17, U7, U8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
